Commit message: add Logger and Arm class

File: config/urdf/yandy_urdf.urdf (robot description, URDF)
Before this commit: robot yandy_urdf, 6 links, 5 joints
Joints:
- joint joint_1: limit lower=0 upper=0 effort=0 velocity=0 -> lower=-2.4 upper=2.4 effort=50 velocity=8
- joint joint_2: limit lower=0 upper=0 effort=0 velocity=0 -> lower=0 upper=2.7 effort=50 velocity=8
- joint joint_3: limit lower=0 upper=0 effort=0 velocity=0 -> lower=-3.2 upper=0 effort=50 velocity=8
- joint joint_4: limit lower=0 upper=0 effort=0 velocity=0 -> effort=50 velocity=8; type revolute -> continuous
- joint joint_5: limit lower=0 upper=0 effort=0 velocity=0 -> lower=0 upper=3.14 effort=50 velocity=8

Commit message: add DynamicsSolver and example program

File: config/urdf/yandy_urdf.urdf (robot description, URDF)
Before this commit: robot yandy_urdf, 6 links, 5 joints
Joints:
- joint joint_4: limit effort=50 velocity=8 -> lower=-6.28 upper=6.28 effort=50 velocity=8; type continuous -> revolute

Commit message: use tcp link

File: config/urdf/yandy_urdf.urdf (robot description, URDF)
Before this commit: robot yandy_urdf, 6 links, 5 joints
Links:
- added link gripper_tcp, mass 0.001
Joints:
- added joint joint_tcp: type fixed, parent link_5, child gripper_tcp, origin xyz=0.2 0 0.035 rpy=0 0 0

Commit message: add camera frame handling and related transformations in DynamicsSolver

File: config/urdf/yandy_urdf.urdf (robot description, URDF)
Before this commit: robot yandy_urdf, 7 links, 6 joints
Links:
- added link camera_optical_frame
Joints:
- added joint camera_joint: type fixed, parent link_3, child camera_optical_frame, origin xyz=0.06 0.18 0.038 rpy=0 -1.5707 3.9269
- joint joint_3: axis 0 0 -1 -> 0 0 1; limit lower=-3.2 upper=0 effort=50 velocity=8 -> lower=0 upper=3.2 effort=50 velocity=8

Commit message: fix joint_3 direction

File: config/urdf/yandy_urdf.urdf (robot description, URDF)
Before this commit: robot yandy_urdf, 8 links, 7 joints
Joints:
- joint joint_tcp: limit (none) -> lower=0 upper=0 effort=50 velocity=8

Commit message: add fixed store joint in urdf

File: config/urdf/yandy_urdf.urdf (robot description, URDF)
Before this commit: robot yandy_urdf, 8 links, 7 joints
Links:
- added link store_frame_1
- added link store_frame_2
Joints:
- added joint store_joint_1: type fixed, parent base_link, child store_frame_1, origin xyz=-0.20 0.22 0.43 rpy=0 0 0
- added joint store_joint_2: type fixed, parent base_link, child store_frame_2, origin xyz=-0.20 -0.27 0.43 rpy=0 0 0

Commit message: new 6dof model loaded

File: config/urdf/yandy_urdf.urdf (robot description, URDF)
Before this commit: robot yandy_urdf, 10 links, 9 joints
Links:
- added link link_6, mass 0.452418521071107; collision mesh filename=meshes/link_6.STL; visual mesh filename=meshes/link_6.STL
Joints:
- added joint joint_6: type revolute, parent link_5, child link_6, origin xyz=0.052 0 0.021 rpy=0 1.5708 0, axis 0 0 -1, limit lower=-6.28 upper=6.28 effort=50 velocity=8
- joint joint_1: axis 0 0 1 -> 0 0 -1; origin xyz=0.0476510115539754 -0.0233859859702091 0.11487414900293 rpy=0 0 0 -> xyz=-2.5649E-05 -1.7585E-05 0.1128 rpy=0 0 0
- joint joint_2: origin xyz=0 -0.0342999999999993 0.0899999999999964 rpy=1.5707963267949 0 3.14159265358979 -> xyz=0 -0.0343 0.114 rpy=1.5708 0 -3.1416
- joint joint_3: origin xyz=0.246201938253051 0.043412044416735 0.0723000000000015 rpy=3.14159265358979 0 -3.14159265358979 -> xyz=0.2462 0.043412 0.0723 rpy=3.1416 0 3.1416
- joint joint_4: axis 0 0 1 -> 0 0 -1; origin xyz=0.142524819154464 0.158289847826683 0.037999999999854 rpy=-1.57079632679561 0 -0.733038285837583 -> xyz=0.13717 0.15234 0.038 rpy=-1.5708 0 -0.73304
- joint joint_5: origin xyz=0 0.034000000000019 0.0599999999999983 rpy=1.5707963267949 0 0 -> xyz=0 0.021 0.068 rpy=1.5708 0 0
- joint joint_tcp: parent link_5 -> link_6; type fixed -> revolute
- joint store_joint_1: origin xyz=-0.20 0.22 0.43 rpy=0 0 0 -> xyz=-0.25 0.25 0.45 rpy=0 0 0
- joint store_joint_2: origin xyz=-0.20 -0.27 0.43 rpy=0 0 0 -> xyz=-0.25 -0.25 0.45 rpy=0 0 0

Commit message: using new 6-dof arm in program

File: config/urdf/yandy_urdf.urdf (robot description, URDF)
Before this commit: robot yandy_urdf, 11 links, 10 joints
Joints:
- joint joint_tcp: limit lower=0 upper=0 effort=50 velocity=8 -> (none); origin xyz=0.2 0 0.035 rpy=0 0 0 -> xyz=0 0 0.12 rpy=0 0 0; type revolute -> fixed
- joint store_joint_1: origin xyz=-0.25 0.25 0.45 rpy=0 0 0 -> xyz=-0.25 0.25 0.6 rpy=-2.3 1.56 0
- joint store_joint_2: origin xyz=-0.25 -0.25 0.45 rpy=0 0 0 -> xyz=-0.25 -0.25 0.6 rpy=2.3 1.56 0

Commit message: use callback function when FSM transition triggered

File: config/urdf/yandy_urdf.urdf (robot description, URDF)
Before this commit: robot yandy_urdf, 11 links, 10 joints
Joints:
- joint store_joint_1: origin xyz=-0.25 0.25 0.6 rpy=-2.3 1.56 0 -> xyz=-0.25 0.25 0.65 rpy=-2.3 1.56 0
- joint store_joint_2: origin xyz=-0.25 -0.25 0.6 rpy=2.3 1.56 0 -> xyz=-0.25 -0.25 0.65 rpy=2.3 1.56 0

Commit message: add gimbal links

File: config/urdf/yandy_urdf.urdf (robot description, URDF)
Before this commit: robot yandy_urdf, 11 links, 10 joints
Links:
- added link gimbal_link_1, mass 0.28493; collision mesh filename=meshes/gimbal_link_1.STL; visual mesh filename=meshes/gimbal_link_1.STL
- added link gimbal_link_2, mass 0.015494; collision mesh filename=meshes/gimbal_link_2.STL; visual mesh filename=meshes/gimbal_link_2.STL
- added link gimbal_link_3, mass 0.065739; collision mesh filename=meshes/gimbal_link_3.STL; visual mesh filename=meshes/gimbal_link_3.STL
- link base_link: mass 5.66689591232295 -> 5.67931087390506
- link link_1: mass 1.44819766694536 -> 0.80797
- link link_2: mass 1.01543198954596 -> 1.0154
- link link_3: mass 1.3087461829584 -> 1.3016
- link link_4: mass 0.479732829832372 -> 0.479732876616794
- link link_5: mass 0.829074880083356 -> 0.563264780449047
Joints:
- added joint gimbal_joint_1: type prismatic, parent link_1, child gimbal_link_1, origin xyz=0.031 0.06 0.0298 rpy=0 0 0, axis 0 0 1, limit lower=0 upper=0.2 effort=50 velocity=8
- added joint gimbal_joint_2: type revolute, parent gimbal_link_1, child gimbal_link_2, origin xyz=0.01505 0.037 0.2921 rpy=0 0 0, axis 0 0 1, limit lower=-2.0 upper=2.0 effort=50 velocity=8
- added joint gimbal_joint_3: type revolute, parent gimbal_link_2, child gimbal_link_3, origin xyz=0.007 -0.023 0.0227 rpy=1.5708 0 0, axis 0 0 1, limit lower=-0.3 upper=0.5 effort=50 velocity=8

Commit message: update fetch method

File: config/urdf/yandy_urdf.urdf (robot description, URDF)
Before this commit: robot yandy_urdf, 14 links, 13 joints
Joints:
- joint joint_6: limit lower=-6.28 upper=6.28 effort=50 velocity=8 -> lower=-3.14 upper=3.14 effort=50 velocity=8

Commit message: add extracting process for store/fetch process

File: config/urdf/yandy_urdf.urdf (robot description, URDF)
Before this commit: robot yandy_urdf, 14 links, 13 joints
Joints:
- joint store_joint_1: origin xyz=-0.25 0.25 0.65 rpy=-2.3 1.56 0 -> xyz=-0.25 0.25 0.40 rpy=-3.0 1.56 0
- joint store_joint_2: origin xyz=-0.25 -0.25 0.65 rpy=2.3 1.56 0 -> xyz=-0.25 -0.25 0.40 rpy=3.0 1.56 0

Commit message: debugging on the car...

File: config/urdf/yandy_urdf.urdf (robot description, URDF)
Before this commit: robot yandy_urdf, 14 links, 13 joints
Links:
- link base_link: mass 5.67931087390506 -> 6.67931087390506
- link link_1: mass 0.80797 -> 2.50797
- link link_2: mass 1.0154 -> 5.5154
- link link_3: mass 1.3016 -> 4.1116
- link link_4: mass 0.479732876616794 -> 1.579732876616794
- link link_5: mass 0.563264780449047 -> 2.063264780449047
- link link_6: mass 0.452418521071107 -> 1.952418521071107

Commit message: update urdf param

File: config/urdf/yandy_urdf.urdf (robot description, URDF)
Before this commit: robot yandy_urdf, 14 links, 13 joints
Links:
- link link_1: mass 2.50797 -> 2.00797
- link link_2: mass 5.5154 -> 5.1154
- link link_3: mass 4.1116 -> 0.7116
- link link_4: mass 1.579732876616794 -> 0.579732876616794
- link link_5: mass 2.063264780449047 -> 0.563264780449047
- link link_6: mass 1.952418521071107 -> 0.752418521071107
Joints:
- joint joint_2: limit lower=0 upper=2.7 effort=50 velocity=8 -> lower=0 upper=2.25 effort=50 velocity=8
- joint joint_6: limit lower=-3.14 upper=3.14 effort=50 velocity=8 -> lower=-2.14 upper=2.14 effort=50 velocity=8

Commit message: twist param

File: config/urdf/yandy_urdf.urdf (robot description, URDF)
Before this commit: robot yandy_urdf, 14 links, 13 joints
Links:
- link link_2: mass 5.1154 -> 4.5154
- link link_3: mass 0.7116 -> 0.5116
- link link_4: mass 0.579732876616794 -> 0.679732876616794
- link link_5: mass 0.563264780449047 -> 0.863264780449047
- link link_6: mass 0.752418521071107 -> 1.552418521071107

Commit message: 上场版参数！

File: config/urdf/yandy_urdf.urdf (robot description, URDF)
Before this commit: robot yandy_urdf, 14 links, 13 joints
Links:
- link link_1: mass 2.00797 -> 1.50797
- link link_2: mass 4.5154 -> 2.0154
- link link_3: mass 0.5116 -> 1.4116
- link link_5: mass 0.863264780449047 -> 0.563264780449047
- link link_6: mass 1.552418521071107 -> 0.972418521071107

Commit message: 最终上场版

File: config/urdf/yandy_urdf.urdf (robot description, URDF)
Before this commit: robot yandy_urdf, 14 links, 13 joints
Links:
- link link_2: mass 2.0154 -> 2.5154
- link link_3: mass 1.4116 -> 1.2116

Commit message: twist params

File: config/urdf/yandy_urdf.urdf (robot description, URDF)
Before this commit: robot yandy_urdf, 14 links, 13 joints
Links:
- link link_1: mass 1.50797 -> 1.00797
Joints:
- joint store_joint_1: origin xyz=-0.25 0.25 0.40 rpy=-3.0 1.56 0 -> xyz=-0.23 0.23 0.40 rpy=-3.0 1.56 0
- joint store_joint_2: origin xyz=-0.25 -0.25 0.40 rpy=3.0 1.56 0 -> xyz=-0.23 -0.23 0.40 rpy=3.0 1.56 0
